File: KiCAD/RideSyncEmbedded_0.0/RideSyncEmbedded_0.0.kicad_sch (KiCad schematic)
At the start: 26 parts, among them IC1 LTC3108, IC2 LTC3108, Q1 CSD23280F3, T1 PA0185NL, U1 LM66100DCK, U2 LT6106, U3 LT6106

Commit message: call
Parts:
- added C4, C5: 1uF, symbol Device:C
- added C8, C9: 0.1uF, symbol Device:C
- added R7: R, symbol Device:R
- added U4, U5: LM66100DCK, Package_TO_SOT_SMD:SOT-363_SC-70-6, symbol Power_Management:LM66100DCK
- added U6, U7: SiP32431DR3, Package_TO_SOT_SMD:SOT-363_SC-70-6, symbol Power_Management:SiP32431DR3
Connections:
- net GND: now also C4.2, C5.2, C8.2, C9.2, U4.2 (GND), U5.2 (GND), U6.2 (GND), U6.5 (GND), U7.2 (GND), U7.5 (GND)
- net Vout: now also C8.1, C9.1, U4.6 (VOUT), U5.6 (VOUT), U6.1 (OUT), U7.1 (OUT)
- net at R2.1, R_sense.2, U1.1 (VIN)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: now also C4.1, R7.1, U4.1 (VIN), U6.3 (ON), U6.4 (IN)
- net V_teg: now reaches C_out.1, IC1.4 (VOUT), R4.2, R_sense.1, U2.5 (V+)
- net V_sun: now reaches C_out1.1, IC2.4 (VOUT), R5.2, R_sense1.1, U3.5 (V+)
- net at Q1.2 (S), R_sense1.2, U1.3 (~{CE})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: now also C5.1, U4.3 (~{CE}), U5.1 (VIN), U7.3 (ON), U7.4 (IN)
- new net: R7.2, U4.5 (ST), U5.3 (~{CE})
Other:
- note added: "Load Switch with Reverse Blocking"
- moved on the sheet: C1, C2, C3, C6, C7, C_out, C_out1, C_store, C_store1, IC1, IC2, PE1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
