File: KiCAD/RideSyncEmbedded_1.0/RideSyncEmbedded_1.2.kicad_sch (KiCad schematic)
At the start: 52 parts, among them IC1 LTC3108, IC2 SIP32431DR3-T1GE3, IC3 MAX40018ATA+, IC4 SIP32431DR3-T1GE3, IC5 INA190A4QDCKRQ1, IC6 MAX40018ATA+, IC7 INA190A4QDCKRQ1, J1 Conn_01x02_Pin, J2 Conn_01x02_Pin, T1 LPR6235-752SMRB

Commit message: TEG setup
Parts:
- added JP10: Sun_current, TestPoint:TestPoint_2Pads_Pitch2.54mm_Drill0.8mm, symbol Jumper:Jumper_2_Small_Bridged
- added JP9: TEG_current, TestPoint:TestPoint_2Pads_Pitch2.54mm_Drill0.8mm, symbol Jumper:Jumper_2_Small_Bridged
Connections:
- net Vout: now also JP9.1 (A); no longer IC2.3 (ON/OFF), IC2.4 (IN)
- net at C6.1, C_out2.1, C_out3.1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: now also JP10.1 (A); no longer IC4.3 (ON/OFF), IC4.4 (IN)
- new net: IC2.3 (ON/OFF), IC2.4 (IN), JP9.2 (B)
- new net: IC4.3 (ON/OFF), IC4.4 (IN), JP10.2 (B)
Other:
- moved on the sheet: C1, C3, C5, C_out1, C_store1, IC1, IC2, IC4, JP1, JP2, R1

Commit message: tlv added
Parts:
- JP2: footprint (none) -> Jumper:SolderJumper-3_P1.3mm_Bridged12_RoundedPad1.0x1.5mm_NumberLabels
Changed lines of the file:
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@@
 			)
 		)
-		(property "Footprint" ""
+		(property "Footprint" "Jumper:SolderJumper-3_P1.3mm_Bridged12_RoundedPad1.0x1.5mm_NumberLabels"
 			(at 140.97 57.15 0)
 			(effects
