File: KiCAD/RideSyncEmbedded_1.0/RideSyncEmbedded_1.4.kicad_sch (KiCad schematic)
At the start: 77 parts, among them IC1 LTC3108, IC2 SIP32431DR3-T1GE3, IC3 MAX40018ATA+, IC4 SIP32432DR3-T1GE3, IC5 INA190A4QDCKRQ1, IC6 MAX40018ATA+, IC7 INA190A4QDCKRQ1, IC8 MAX40018ATA+, IC9 MAX40018ATA+, J1 Conn_01x02_Pin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

Commit message: jpg assets
Parts:
- R13: value 3.3M -> 4.7M
- R14: value 5.76M -> 8.2M
Changed lines of the file:
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@@
 			)
 		)
-		(property "Value" "3.3M"
+		(property "Value" "4.7M"
 			(at 81.28 96.52 90)
 			(effects
@@
 			)
 		)
-		(property "Value" "5.76M"
+		(property "Value" "8.2M"
 			(at 91.44 96.52 90)
 			(effects
