File: KiCAD/RideSyncEmbedded_2.0/RideSyncEmbedded_2.0.kicad_sch (KiCad schematic)
At the start: 76 parts, among them IC2 SIP32431DR3-T1GE3, IC3 MAX40018ATA+, IC4 SIP32432DR3-T1GE3, IC5 INA190A4QDCKRQ1, IC6 MAX40018ATA+, IC7 INA190A4QDCKRQ1, IC8 MAX40018ATA+, IC9 MAX40018ATA+, J1 Conn_01x02_Pin, J2 Conn_01x02_Pin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

Commit message: fianl results ppt
Parts:
- C_store1: value 0.022F -> 0.021F
Changed lines of the file:
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@@
 			)
 		)
-		(property "Value" "0.022F"
+		(property "Value" "0.021F"
 			(at 189.23 34.9249 0)
 			(effects

Commit message: fig
Parts:
- removed IC6: MAX40018ATA+, SON65P300X300X80-9N, symbol MAX40018ATA+:MAX40018ATA+
- removed R2, R3, R4, R5, R6, R7, R8, R9: R, symbol Device:R
Connections:
- no-connect marks 24 -> 23
Other:
- note removed: "MAX40018 | Discrete current measurement: VOUT = R3/R2(V1-V2)"
- moved on the sheet: H1, H2, H3, IC5, IC7, J1, J2, JP3, JP4, JP5, JP6, JP7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

Commit message: schema
Parts:
- C7: value C_load -> C_out
- renumbered C_store2 to C_PV, C_store1 to C_TEG
Changed lines of the file:
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@@
 		(dnp no)
 		(fields_autoplaced yes)
-		(property "Reference" "C_store2"
+		(property "Reference" "C_PV"
 			(at 170.18 80.6449 0)
 			(effects
@@
 			(project "RideSyncEmbedded_1.4"
 				(path "/2814c729-d4e6-4af1-8503-05b33a930358"
-					(reference "C_store2")
+					(reference "C_PV")
 					(unit 1)
 				)
@@
 		(dnp no)
 		(fields_autoplaced yes)
-		(property "Reference" "C_store1"
+		(property "Reference" "C_TEG"
 			(at 189.23 32.3849 0)
 			(effects
@@
 			(project "RideSyncEmbedded_2.0"
 				(path "/2814c729-d4e6-4af1-8503-05b33a930358"
-					(reference "C_store1")
+					(reference "C_TEG")
 					(unit 1)
 				)
@@
 			)
 		)
-		(property "Value" "C_load"
+		(property "Value" "C_out"
 			(at 275.59 39.3699 0)
 			(effects
